Commit message: updated isaac and description

File: cerberus_ws/install/cerberus_description/share/cerberus_description/urdf/cerberus_odrive.urdf.xacro (robot description, xacro)
@@ -1,167 +1 @@
-<?xml version="1.0"?>
-<robot xmlns:xacro="http://www.ros.org/wiki/xacro" name="odrive_robot">
-  <!-- Arguments controlling whether each of the 12 joints is enabled -->
-  <xacro:arg name="enable_joint0"  default="false" />
-  <xacro:arg name="enable_joint1"  default="false" />
-  <xacro:arg name="enable_joint2"  default="false" />
-  <xacro:arg name="enable_joint3"  default="false" />
-  <xacro:arg name="enable_joint4"  default="false" />
-  <xacro:arg name="enable_joint5"  default="false" />
-  <xacro:arg name="enable_joint6"  default="false" />
-  <xacro:arg name="enable_joint7"  default="false" />
-  <xacro:arg name="enable_joint8"  default="false" />
-  <xacro:arg name="enable_joint9"  default="false" />
-  <xacro:arg name="enable_joint10" default="false" />
-  <xacro:arg name="enable_joint11" default="false" />
-  <!-- Arguments for up to 6 ODrive boards (2 axes each) -->
-  <xacro:arg name="odrive_1_serial" default="2081356E524B" />
-  <xacro:arg name="odrive_2_serial" default="20763599524B" />
-  <xacro:arg name="odrive_3_serial" default="000000000000" />
-  <xacro:arg name="odrive_4_serial" default="000000000000" />
-  <xacro:arg name="odrive_5_serial" default="000000000000" />
-  <xacro:arg name="odrive_6_serial" default="000000000000" />
-  <!-- Include your custom ODrive xacro definition that handles up to two axes -->
-  <xacro:include filename="$(find cerberus_description)/urdf/odrive.ros2_control.xacro" />
-  <!-- A world link to anchor everything -->
-  <link name="world" />
-  <!-- Define 12 links and 12 joints, each optional behind an enable_jointN check -->
-  <xacro:if value="$(arg enable_joint0)">
-    <link name="link0" />
-    <joint name="joint0" type="continuous">
-      <parent link="world"/>
-      <child link="link0"/>
-      <axis xyz="0 0 1"/>
-    </joint>
-  </xacro:if>
-  <xacro:if value="$(arg enable_joint1)">
-    <link name="link1" />
-    <joint name="joint1" type="continuous">
-      <parent link="world"/>
-      <child link="link1"/>
-      <axis xyz="0 0 1"/>
-    </joint>
-  </xacro:if>
-  <xacro:if value="$(arg enable_joint2)">
-    <link name="link2" />
-    <joint name="joint2" type="continuous">
-      <parent link="world"/>
-      <child link="link2"/>
-      <axis xyz="0 0 1"/>
-    </joint>
-  </xacro:if>
-  <xacro:if value="$(arg enable_joint3)">
-    <link name="link3" />
-    <joint name="joint3" type="continuous">
-      <parent link="world"/>
-      <child link="link3"/>
-      <axis xyz="0 0 1"/>
-    </joint>
-  </xacro:if>
-  <xacro:if value="$(arg enable_joint4)">
-    <link name="link4" />
-    <joint name="joint4" type="continuous">
-      <parent link="world"/>
-      <child link="link4"/>
-      <axis xyz="0 0 1"/>
-    </joint>
-  </xacro:if>
-  <xacro:if value="$(arg enable_joint5)">
-    <link name="link5" />
-    <joint name="joint5" type="continuous">
-      <parent link="world"/>
-      <child link="link5"/>
-      <axis xyz="0 0 1"/>
-    </joint>
-  </xacro:if>
-  <xacro:if value="$(arg enable_joint6)">
-    <link name="link6" />
-    <joint name="joint6" type="continuous">
-      <parent link="world"/>
-      <child link="link6"/>
-      <axis xyz="0 0 1"/>
-    </joint>
-  </xacro:if>
-  <xacro:if value="$(arg enable_joint7)">
-    <link name="link7" />
-    <joint name="joint7" type="continuous">
-      <parent link="world"/>
-      <child link="link7"/>
-      <axis xyz="0 0 1"/>
-    </joint>
-  </xacro:if>
-  <xacro:if value="$(arg enable_joint8)">
-    <link name="link8" />
-    <joint name="joint8" type="continuous">
-      <parent link="world"/>
-      <child link="link8"/>
-      <axis xyz="0 0 1"/>
-    </joint>
-  </xacro:if>
-  <xacro:if value="$(arg enable_joint9)">
-    <link name="link9" />
-    <joint name="joint9" type="continuous">
-      <parent link="world"/>
-      <child link="link9"/>
-      <axis xyz="0 0 1"/>
-    </joint>
-  </xacro:if>
-  <xacro:if value="$(arg enable_joint10)">
-    <link name="link10" />
-    <joint name="joint10" type="continuous">
-      <parent link="world"/>
-      <child link="link10"/>
-      <axis xyz="0 0 1"/>
-    </joint>
-  </xacro:if>
-  <xacro:if value="$(arg enable_joint11)">
-    <link name="link11" />
-    <joint name="joint11" type="continuous">
-      <parent link="world"/>
-      <child link="link11"/>
-      <axis xyz="0 0 1"/>
-    </joint>
-  </xacro:if>
-  <!-- Now define 6 possible ODrive boards, each controlling 2 joints -->
-  <!-- ODrive #1: controls joint0 and joint1 -->
-  <xacro:odrive_ros2_control
-    name="odrive1_ros2_control"
-    sensor_name="odrv0"
-    serial_number="$(arg odrive_1_serial)"
-    joint0_name="joint0" enable_joint0="$(arg enable_joint0)"
-    joint1_name="joint1" enable_joint1="$(arg enable_joint1)" />
-  <!-- ODrive #2: controls joint2 and joint3 -->
-  <xacro:odrive_ros2_control
-    name="odrive2_ros2_control"
-    sensor_name="odrv1"
-    serial_number="$(arg odrive_2_serial)"
-    joint0_name="joint2" enable_joint0="$(arg enable_joint2)"
-    joint1_name="joint3" enable_joint1="$(arg enable_joint3)" />
-  <!-- ODrive #3: controls joint4 and joint5 -->
-  <xacro:odrive_ros2_control
-    name="odrive3_ros2_control"
-    sensor_name="odrv2"
-    serial_number="$(arg odrive_3_serial)"
-    joint0_name="joint4" enable_joint0="$(arg enable_joint4)"
-    joint1_name="joint5" enable_joint1="$(arg enable_joint5)" />
-  <!-- ODrive #4: controls joint6 and joint7 -->
-  <xacro:odrive_ros2_control
-    name="odrive4_ros2_control"
-    sensor_name="odrv3"
-    serial_number="$(arg odrive_4_serial)"
-    joint0_name="joint6" enable_joint0="$(arg enable_joint6)"
-    joint1_name="joint7" enable_joint1="$(arg enable_joint7)" />
-  <!-- ODrive #5: controls joint8 and joint9 -->
-  <xacro:odrive_ros2_control
-    name="odrive5_ros2_control"
-    sensor_name="odrv4"
-    serial_number="$(arg odrive_5_serial)"
-    joint0_name="joint8" enable_joint0="$(arg enable_joint8)"
-    joint1_name="joint9" enable_joint1="$(arg enable_joint9)" />
-  <!-- ODrive #6: controls joint10 and joint11 -->
-  <xacro:odrive_ros2_control
-    name="odrive6_ros2_control"
-    sensor_name="odrv5"
-    serial_number="$(arg odrive_6_serial)"
-    joint0_name="joint10" enable_joint0="$(arg enable_joint10)"
-    joint1_name="joint11" enable_joint1="$(arg enable_joint11)" />
-</robot>
+/home/v/Dev/Github/Cerberus/Control/cerberus_ws/src/cerberus_final/cerberus_description/urdf/cerberus_odrive.urdf.xacro

File: cerberus_ws/install/cerberus_description/share/cerberus_description/urdf/cerberus_two_odrive.urdf.xacro (robot description, xacro)
@@ -1,35 +1 @@
-<?xml version="1.0"?>
-<robot xmlns:xacro="http://www.ros.org/wiki/xacro" name="odrive_robot">
-  <!-- Arguments controlling whether each of the 12 joints is enabled -->
-  <xacro:arg name="enable_joint0"  default="false" />
-  <xacro:arg name="enable_joint1"  default="false" />
-  <!-- Arguments for up to 6 ODrive boards (2 axes each) -->
-  <xacro:arg name="odrive_1_serial" default="2081356E524B" />
-  <!-- Include your custom ODrive xacro definition that handles up to two axes -->
-  <xacro:include filename="$(find cerberus_description)/urdf/odrive.ros2_control.xacro" />
-  <!-- A world link to anchor everything -->
-  <link name="world" />
-  <!-- Define 12 links and 12 joints, each optional behind an enable_jointN check -->
-  <xacro:if value="$(arg enable_joint0)">
-    <link name="link0" />
-    <joint name="joint0" type="continuous">
-      <parent link="world"/>
-      <child link="link0"/>
-      <axis xyz="0 0 1"/>
-    </joint>
-  </xacro:if>
-  <xacro:if value="$(arg enable_joint1)">
-    <link name="link1" />
-    <joint name="joint1" type="continuous">
-      <parent link="world"/>
-      <child link="link1"/>
-      <axis xyz="0 0 1"/>
-    </joint>
-  </xacro:if>
-  <xacro:odrive_ros2_control
-    name="odrive1_ros2_control"
-    sensor_name="odrv0"
-    serial_number="$(arg odrive_1_serial)"
-    joint0_name="joint0" enable_joint0="$(arg enable_joint0)"
-    joint1_name="joint1" enable_joint1="$(arg enable_joint1)" />
-</robot>
+/home/v/Dev/Github/Cerberus/Control/cerberus_ws/src/cerberus_final/cerberus_description/urdf/cerberus_two_odrive.urdf.xacro

File: cerberus_ws/install/cerberus_description/share/cerberus_description/urdf/cerbiboi.urdf.xacro (robot description, xacro)
@@ -1,168 +1 @@
-<?xml version="1.0"?>
-<robot xmlns:xacro="http://www.ros.org/wiki/xacro" name="Cerberus">
-    <xacro:include filename="$(find cerberus_description)/urdf/leg_macro.xacro" />
-    <!--
-    <link name="world" />
-    <joint name="world_joint" type="fixed">
-        <parent link="world" />
-        <child link="base_link" />
-    </joint>
-    -->
-    <link name="base_link">
-        <visual>
-            <geometry>
-                <box size="0.6 0.282 0.2" />
-            </geometry>
-            <material name="blue">
-                <color rgba="0.3 0.3 0.8 1.0" />
-            </material>
-        </visual>
-        <collision>
-            <geometry>
-                <box size="0.6 0.282 0.2" />
-            </geometry>
-        </collision>
-        <inertial>
-            <mass value="5.0" />
-            <inertia ixx="0.0833" iyy="0.1667" izz="0.2167"
-                ixy="0.0" ixz="0.0" iyz="0.0" />
-        </inertial>
-    </link>
-    <xacro:leg_macro
-        leg_name="front_left"
-        parent_link="base_link"
-        gearbox_offset="0.1"
-        connector_xyz="0.35 0.08 0"
-        connector_rpy="0 1.5707963267948966 0"
-    />
-    <xacro:leg_macro
-        leg_name="front_right"
-        parent_link="base_link"
-        gearbox_offset="0.1"
-        connector_xyz="0.35 -0.08 0"
-        connector_rpy="3.14159265 -1.5707963267948966 0"
-    />
-    <xacro:leg_macro
-        leg_name="rear_left"
-        parent_link="base_link"
-        gearbox_offset="-0.1"
-        connector_xyz="-0.35 0.08 0"
-        connector_rpy="0 1.5707963267948966 0"
-    />
-    <xacro:leg_macro
-        leg_name="rear_right"
-        parent_link="base_link"
-        gearbox_offset="-0.1"
-        connector_xyz="-0.35 -0.08 0"
-        connector_rpy="3.14159265 -1.5707963267948966 0"
-    />
-    <ros2_control name="IgnitionSystem" type="system">
-        <hardware>
-            <plugin>ign_ros2_control/IgnitionSystem</plugin>
-        </hardware>
-        <joint name="front_left_shoulder_connector">
-            <command_interface name="position" />
-            <command_interface name="velocity" />
-            <command_interface name="effort" />
-            <state_interface name="position" />
-            <state_interface name="velocity" />
-            <state_interface name="effort" />
-        </joint>
-        <joint name="front_left_shoulder_leg">
-            <command_interface name="position" />
-            <command_interface name="velocity" />
-            <command_interface name="effort" />
-            <state_interface name="position" />
-            <state_interface name="velocity" />
-            <state_interface name="effort" />
-        </joint>
-        <joint name="front_left_knee">
-            <command_interface name="position" />
-            <command_interface name="velocity" />
-            <command_interface name="effort" />
-            <state_interface name="position" />
-            <state_interface name="velocity" />
-            <state_interface name="effort" />
-        </joint>
-        <joint name="front_right_shoulder_connector">
-            <command_interface name="position" />
-            <command_interface name="velocity" />
-            <command_interface name="effort" />
-            <state_interface name="position" />
-            <state_interface name="velocity" />
-            <state_interface name="effort" />
-        </joint>
-        <joint name="front_right_shoulder_leg">
-            <command_interface name="position" />
-            <command_interface name="velocity" />
-            <command_interface name="effort" />
-            <state_interface name="position" />
-            <state_interface name="velocity" />
-            <state_interface name="effort" />
-        </joint>
-        <joint name="front_right_knee">
-            <command_interface name="position" />
-            <command_interface name="velocity" />
-            <command_interface name="effort" />
-            <state_interface name="position" />
-            <state_interface name="velocity" />
-            <state_interface name="effort" />
-        </joint>
-        <joint name="rear_left_shoulder_connector">
-            <command_interface name="position" />
-            <command_interface name="velocity" />
-            <command_interface name="effort" />
-            <state_interface name="position" />
-            <state_interface name="velocity" />
-            <state_interface name="effort" />
-        </joint>
-        <joint name="rear_left_shoulder_leg">
-            <command_interface name="position" />
-            <command_interface name="velocity" />
-            <command_interface name="effort" />
-            <state_interface name="position" />
-            <state_interface name="velocity" />
-            <state_interface name="effort" />
-        </joint>
-        <joint name="rear_left_knee">
-            <command_interface name="position" />
-            <command_interface name="velocity" />
-            <command_interface name="effort" />
-            <state_interface name="position" />
-            <state_interface name="velocity" />
-            <state_interface name="effort" />
-        </joint>
-        <joint name="rear_right_shoulder_connector">
-            <command_interface name="position" />
-            <command_interface name="velocity" />
-            <command_interface name="effort" />
-            <state_interface name="position" />
-            <state_interface name="velocity" />
-            <state_interface name="effort" />
-        </joint>
-        <joint name="rear_right_shoulder_leg">
-            <command_interface name="position" />
-            <command_interface name="velocity" />
-            <command_interface name="effort" />
-            <state_interface name="position" />
-            <state_interface name="velocity" />
-            <state_interface name="effort" />
-        </joint>
-        <joint name="rear_right_knee">
-            <command_interface name="position" />
-            <command_interface name="velocity" />
-            <command_interface name="effort" />
-            <state_interface name="position" />
-            <state_interface name="velocity" />
-            <state_interface name="effort" />
-        </joint>
-    </ros2_control>
-    <gazebo>
-        <plugin filename="ign_ros2_control-system"
-            name="ign_ros2_control::IgnitionROS2ControlPlugin">
-            <robot_param>robot_description</robot_param>
-            <robot_param_node>robot_state_publisher</robot_param_node>
-            <parameters>$(find cerberus_bringup)/config/cerberus.yaml</parameters>
-        </plugin>
-    </gazebo>
-</robot>
+/home/v/Dev/Github/Cerberus/Control/cerberus_ws/src/cerberus_final/cerberus_description/urdf/cerbiboi.urdf.xacro

File: cerberus_ws/install/cerberus_description/share/cerberus_description/urdf/leg_macro.xacro (robot description, xacro)
@@ -1,123 +1 @@
-<?xml version="1.0"?>
-<robot xmlns:xacro="http://www.ros.org/wiki/xacro">
-  <xacro:macro name="leg_macro" params="
-      leg_name
-      parent_link
-      gearbox_offset
-      connector_xyz:='0.35 0.08 0'
-      connector_rpy:='0 1.5707963267948966 0'
-    ">
-    <joint name="${leg_name}_leg_connector" type="fixed">
-      <parent link="${parent_link}" />
-      <child link="${leg_name}_gearbox_shoulder" />
-      <origin xyz="${connector_xyz}" rpy="${connector_rpy}" />
-    </joint>
-    <link name="${leg_name}_gearbox_shoulder">
-      <visual>
-        <geometry>
-          <cylinder radius="0.055" length="0.1" />
-        </geometry>
-        <material name="purple">
-          <color rgba="0.43 0.27 0.52 1" />
-        </material>
-      </visual>
-      <collision>
-        <geometry>
-          <cylinder radius="0.055" length="0.1" />
-        </geometry>
-      </collision>
-      <inertial>
-        <mass value="0.8" />
-        <inertia ixx="0.01" iyy="0.01" izz="0.01"
-                 ixy="0" ixz="0" iyz="0" />
-      </inertial>
-    </link>
-    <joint name="${leg_name}_shoulder_connector" type="revolute">
-      <parent link="${leg_name}_gearbox_shoulder" />
-      <child link="${leg_name}_gearbox_shoulder2" />
-      <origin xyz="0 0 ${gearbox_offset}" rpy="1.5707963267948963 0 0" />
-      <axis xyz="0 1 0" />
-      <limit effort="200.0" velocity="2.0" lower="-1.57" upper="1.57" />
-    </joint>
-    <link name="${leg_name}_gearbox_shoulder2">
-      <visual>
-        <origin xyz="0 0 -0.0175" />
-        <geometry>
-          <cylinder radius="0.055" length="0.1" />
-        </geometry>
-        <material name="purple">
-          <color rgba="0.43 0.27 0.52 1" />
-        </material>
-      </visual>
-      <collision>
-        <origin xyz="0 0 -0.0175" />
-        <geometry>
-          <cylinder radius="0.055" length="0.1" />
-        </geometry>
-      </collision>
-      <inertial>
-        <mass value="0.8" />
-        <inertia ixx="0.01" iyy="0.01" izz="0.01"
-                 ixy="0" ixz="0" iyz="0" />
-      </inertial>
-    </link>
-    <joint name="${leg_name}_shoulder_leg" type="revolute">
-      <parent link="${leg_name}_gearbox_shoulder2" />
-      <child link="${leg_name}_upper_leg" />
-      <origin xyz="0 0 -0.138" rpy="1.5707963267948963 0 0" />
-      <axis xyz="0 1 0" />
-      <limit effort="200.0" velocity="2.0" lower="-1.57" upper="1.57" />
-    </joint>
-    <link name="${leg_name}_upper_leg">
-      <visual>
-        <origin xyz="0 0 0.15" />
-        <geometry>
-          <cylinder radius="0.055" length="0.3" />
-        </geometry>
-        <material name="purple">
-          <color rgba="0.43 0.27 0.52 1" />
-        </material>
-      </visual>
-      <collision>
-        <origin xyz="0 0 0.15" />
-        <geometry>
-          <cylinder radius="0.055" length="0.3" />
-        </geometry>
-      </collision>
-      <inertial>
-        <mass value="0.8" />
-        <inertia ixx="0.01" iyy="0.01" izz="0.01"
-                 ixy="0" ixz="0" iyz="0" />
-      </inertial>
-    </link>
-    <joint name="${leg_name}_knee" type="revolute">
-      <parent link="${leg_name}_upper_leg" />
-      <child link="${leg_name}_lower_leg" />
-      <origin xyz="0 0 0.3" rpy="0 0 0" />
-      <axis xyz="0 1 0" />
-      <limit effort="200.0" velocity="2.0" lower="-1.57" upper="1.57" />
-    </joint>
-    <link name="${leg_name}_lower_leg">
-      <visual>
-        <origin xyz="0 0 0.15" />
-        <geometry>
-          <cylinder radius="0.035" length="0.3" />
-        </geometry>
-        <material name="purple">
-          <color rgba="0.43 0.27 0.52 1" />
-        </material>
-      </visual>
-      <collision>
-        <origin xyz="0 0 0.15" />
-        <geometry>
-          <cylinder radius="0.035" length="0.3" />
-        </geometry>
-      </collision>
-      <inertial>
-        <mass value="0.8" />
-        <inertia ixx="0.01" iyy="0.01" izz="0.01"
-                 ixy="0" ixz="0" iyz="0" />
-      </inertial>
-    </link>
-  </xacro:macro>
-</robot>
+/home/v/Dev/Github/Cerberus/Control/cerberus_ws/src/cerberus_final/cerberus_description/urdf/leg_macro.xacro

File: cerberus_ws/install/cerberus_description/share/cerberus_description/urdf/odrive.ros2_control.xacro (robot description, xacro)
@@ -1,30 +1 @@
-<?xml version="1.0"?>
-<robot xmlns:xacro="http://www.ros.org/wiki/xacro">
-  <xacro:macro name="odrive_ros2_control"
-    params="name sensor_name serial_number:=^|000000000000 enable_joint0:=^|true enable_joint1:=^|true joint0_name:=^|joint0 joint1_name:=^|joint1">
-    <ros2_control name="${name}" type="system">
-      <hardware>
-        <plugin>odrive_hardware_interface/ODriveHardwareInterface</plugin>
-      </hardware>
-      <sensor name="${sensor_name}">
-        <param name="serial_number">${serial_number}</param>
-      </sensor>
-      <xacro:if value="${enable_joint0}">
-        <joint name="${joint0_name}">
-          <param name="serial_number">${serial_number}</param>
-          <param name="axis">0</param>
-          <param name="enable_watchdog">0</param>
-          <param name="watchdog_timeout">0.0</param>
-        </joint>
-      </xacro:if>
-      <xacro:if value="${enable_joint1}">
-        <joint name="${joint1_name}">
-          <param name="serial_number">${serial_number}</param>
-          <param name="axis">1</param>
-          <param name="enable_watchdog">0</param>
-          <param name="watchdog_timeout">0.0</param>
-        </joint>
-      </xacro:if>
-    </ros2_control>
-  </xacro:macro>
-</robot>
+/home/v/Dev/Github/Cerberus/Control/cerberus_ws/src/cerberus_final/cerberus_description/urdf/odrive.ros2_control.xacro
