Commit message: updated isaac and description

File: cerberus_ws/src/cerberus_final/cerberus_description/urdf/cerbiboi.urdf.xacro (robot description, xacro)
@@ -2,4 +2,6 @@
 <robot xmlns:xacro="http://www.ros.org/wiki/xacro" name="Cerberus">
     <xacro:include filename="$(find cerberus_description)/urdf/leg_macro.xacro" />
+    <xacro:arg name="effort" default="20" />
+    <xacro:arg name="max_joint_velocity" default="150.0" />
     <!--
     <link name="world" />
@@ -12,5 +14,5 @@
         <visual>
             <geometry>
-                <box size="0.6 0.282 0.2" />
+                <box size="0.45 0.282 0.2" />
             </geometry>
             <material name="blue">
@@ -20,10 +22,10 @@
         <collision>
             <geometry>
-                <box size="0.6 0.282 0.2" />
+                <box size="0.45 0.282 0.2" />
             </geometry>
         </collision>
         <inertial>
             <mass value="5.0" />
-            <inertia ixx="0.0833" iyy="0.1667" izz="0.2167"
+            <inertia ixx="0.04980166667" iyy="0.1010416667" izz="0.11751"
                 ixy="0.0" ixz="0.0" iyz="0.0" />
         </inertial>
@@ -33,6 +35,15 @@
         parent_link="base_link"
         gearbox_offset="0.1"
-        connector_xyz="0.35 0.08 0"
+        connector_xyz="0.275 0.08 0"
         connector_rpy="0 1.5707963267948966 0"
+        axis="0 1 0"
+        rot_off="1.5707963267948966"
+        shoulder_lower_limit="-2.094395102"
+        shoulder_upper_limit="1.047197551"
+        knee_rot_off="1.5707963267948966"
+        knee_lower_limit="-0.5235987756"
+        knee_upper_limit="1.047197551"
+        effort="$(arg effort)"
+        max_joint_velocity="$(arg effort)"
     />
     <xacro:leg_macro
@@ -40,6 +51,15 @@
         parent_link="base_link"
         gearbox_offset="0.1"
-        connector_xyz="0.35 -0.08 0"
+        connector_xyz="0.275 -0.08 0"
         connector_rpy="3.14159265 -1.5707963267948966 0"
+        axis="0 -1 0"
+        rot_off="-1.5707963267948966"
+        shoulder_lower_limit="-2.094395102"
+        shoulder_upper_limit="1.047197551"
+        knee_rot_off="-1.5707963267948966"
+        knee_lower_limit="-0.5235987756"
+        knee_upper_limit="1.047197551"
+        effort="$(arg effort)"
+        max_joint_velocity="$(arg effort)"
     />
     <xacro:leg_macro
@@ -47,6 +67,15 @@
         parent_link="base_link"
         gearbox_offset="-0.1"
-        connector_xyz="-0.35 0.08 0"
+        connector_xyz="-0.275 0.08 0"
         connector_rpy="0 1.5707963267948966 0"
+        axis="0 1 0"
+        rot_off="1.5707963267948966"
+        shoulder_lower_limit="-2.094395102"
+        shoulder_upper_limit="1.047197551"
+        knee_rot_off="1.5707963267948966"
+        knee_lower_limit="-0.5235987756"
+        knee_upper_limit="1.047197551"
+        effort="$(arg effort)"
+        max_joint_velocity="$(arg effort)"
     />
     <xacro:leg_macro
@@ -54,6 +83,15 @@
         parent_link="base_link"
         gearbox_offset="-0.1"
-        connector_xyz="-0.35 -0.08 0"
+        connector_xyz="-0.275 -0.08 0"
         connector_rpy="3.14159265 -1.5707963267948966 0"
+        axis="0 -1 0"
+        rot_off="-1.5707963267948966"
+        shoulder_lower_limit="-2.094395102"
+        shoulder_upper_limit="1.047197551"
+        knee_rot_off="-1.5707963267948966"
+        knee_lower_limit="-0.5235987756"
+        knee_upper_limit="1.047197551"
+        effort="$(arg effort)"
+        max_joint_velocity="$(arg effort)"
     />
     <ros2_control name="IgnitionSystem" type="system">
@@ -64,96 +102,72 @@
             <command_interface name="position" />
             <command_interface name="velocity" />
-            <command_interface name="effort" />
             <state_interface name="position" />
             <state_interface name="velocity" />
-            <state_interface name="effort" />
         </joint>
         <joint name="front_left_shoulder_leg">
             <command_interface name="position" />
             <command_interface name="velocity" />
-            <command_interface name="effort" />
             <state_interface name="position" />
             <state_interface name="velocity" />
-            <state_interface name="effort" />
         </joint>
         <joint name="front_left_knee">
             <command_interface name="position" />
             <command_interface name="velocity" />
-            <command_interface name="effort" />
             <state_interface name="position" />
             <state_interface name="velocity" />
-            <state_interface name="effort" />
         </joint>
         <joint name="front_right_shoulder_connector">
             <command_interface name="position" />
             <command_interface name="velocity" />
-            <command_interface name="effort" />
             <state_interface name="position" />
             <state_interface name="velocity" />
-            <state_interface name="effort" />
         </joint>
         <joint name="front_right_shoulder_leg">
             <command_interface name="position" />
             <command_interface name="velocity" />
-            <command_interface name="effort" />
             <state_interface name="position" />
             <state_interface name="velocity" />
-            <state_interface name="effort" />
         </joint>
         <joint name="front_right_knee">
             <command_interface name="position" />
             <command_interface name="velocity" />
-            <command_interface name="effort" />
             <state_interface name="position" />
             <state_interface name="velocity" />
-            <state_interface name="effort" />
         </joint>
         <joint name="rear_left_shoulder_connector">
             <command_interface name="position" />
             <command_interface name="velocity" />
-            <command_interface name="effort" />
             <state_interface name="position" />
             <state_interface name="velocity" />
-            <state_interface name="effort" />
         </joint>
         <joint name="rear_left_shoulder_leg">
             <command_interface name="position" />
             <command_interface name="velocity" />
-            <command_interface name="effort" />
             <state_interface name="position" />
             <state_interface name="velocity" />
-            <state_interface name="effort" />
         </joint>
         <joint name="rear_left_knee">
             <command_interface name="position" />
             <command_interface name="velocity" />
-            <command_interface name="effort" />
             <state_interface name="position" />
             <state_interface name="velocity" />
-            <state_interface name="effort" />
         </joint>
         <joint name="rear_right_shoulder_connector">
             <command_interface name="position" />
             <command_interface name="velocity" />
-            <command_interface name="effort" />
             <state_interface name="position" />
             <state_interface name="velocity" />
-            <state_interface name="effort" />
         </joint>
         <joint name="rear_right_shoulder_leg">
             <command_interface name="position" />
             <command_interface name="velocity" />
-            <command_interface name="effort" />
             <state_interface name="position" />
             <state_interface name="velocity" />
-            <state_interface name="effort" />
         </joint>
         <joint name="rear_right_knee">
             <command_interface name="position" />
             <command_interface name="velocity" />
-            <command_interface name="effort" />
             <state_interface name="position" />
             <state_interface name="velocity" />
-            <state_interface name="effort" />
         </joint>
     </ros2_control>
@@ -166,3 +180,16 @@
         </plugin>
     </gazebo>
+    <gazebo reference="base_link">
+        <sensor name="imu_sensor" type="imu">
+            <!-- Typically you need some sub-elements under <imu> -->
+            <update_rate>50</update_rate>
+            <always_on>true</always_on>
+            <visualize>true</visualize>
+            <topic>imu</topic>
+            <imu>
+                <noise type="none" />
+                <!-- or define noise parameters here -->
+            </imu>
+        </sensor>
+    </gazebo>
 </robot>

File: cerberus_ws/src/cerberus_final/cerberus_description/urdf/leg_macro.xacro (robot description, xacro)
@@ -1,5 +1,6 @@
 <?xml version="1.0"?>
 <robot xmlns:xacro="http://www.ros.org/wiki/xacro">
-  <xacro:macro name="leg_macro" params="
+  <xacro:macro name="leg_macro"
+    params="
       leg_name
       parent_link
@@ -7,4 +8,13 @@
       connector_xyz:='0.35 0.08 0'
       connector_rpy:='0 1.5707963267948966 0'
+      axis:='0 1 0'
+      rot_off='0'
+      shoulder_lower_limit='-1.57'
+      shoulder_upper_limit='1.57'
+      knee_rot_off='0'
+      knee_lower_limit='-1.57'
+      knee_upper_limit='1.57'
+      effort='200'
+      max_joint_velocity='2.0'
     ">
     <joint name="${leg_name}_leg_connector" type="fixed">
@@ -28,7 +38,7 @@
       </collision>
       <inertial>
-        <mass value="0.8" />
-        <inertia ixx="0.01" iyy="0.01" izz="0.01"
-                 ixy="0" ixz="0" iyz="0" />
+        <mass value="0.95" />
+        <inertia ixx="0.01" iyy="0.01" izz="0.01"
+          ixy="0" ixz="0" iyz="0" />
       </inertial>
     </link>
@@ -37,6 +47,6 @@
       <child link="${leg_name}_gearbox_shoulder2" />
       <origin xyz="0 0 ${gearbox_offset}" rpy="1.5707963267948963 0 0" />
-      <axis xyz="0 1 0" />
-      <limit effort="200.0" velocity="2.0" lower="-1.57" upper="1.57" />
+      <axis xyz="${axis}" />
+      <limit effort="${effort}" velocity="${max_joint_velocity}" lower="-1.57" upper="1.57" />
     </joint>
     <link name="${leg_name}_gearbox_shoulder2">
@@ -57,7 +67,7 @@
       </collision>
       <inertial>
-        <mass value="0.8" />
-        <inertia ixx="0.01" iyy="0.01" izz="0.01"
-                 ixy="0" ixz="0" iyz="0" />
+        <mass value="0.95" />
+        <inertia ixx="0.01" iyy="0.01" izz="0.01"
+          ixy="0" ixz="0" iyz="0" />
       </inertial>
     </link>
@@ -65,7 +75,35 @@
       <parent link="${leg_name}_gearbox_shoulder2" />
       <child link="${leg_name}_upper_leg" />
-      <origin xyz="0 0 -0.138" rpy="1.5707963267948963 0 0" />
-      <axis xyz="0 1 0" />
-      <limit effort="200.0" velocity="2.0" lower="-1.57" upper="1.57" />
+      <origin xyz="0 0 -0.1205" rpy="1.5707963267948963 0 ${rot_off}" />
+      <axis xyz="${axis}" />
+      <limit effort="${effort}" velocity="${max_joint_velocity}" lower="${shoulder_lower_limit}"
+        upper="${shoulder_upper_limit}" />
+    </joint>
+    <link name="${leg_name}_outer_gearbox">
+      <visual>
+        <origin xyz="0 0 -0.0175" />
+        <geometry>
+          <cylinder radius="0.055" length="0.1" />
+        </geometry>
+        <material name="purple">
+          <color rgba="0.43 0.27 0.52 1" />
+        </material>
+      </visual>
+      <collision>
+        <origin xyz="0 0 -0.0175" />
+        <geometry>
+          <cylinder radius="0.055" length="0.1" />
+        </geometry>
+      </collision>
+      <inertial>
+        <mass value="0.95" />
+        <inertia ixx="0.01" iyy="0.01" izz="0.01"
+          ixy="0" ixz="0" iyz="0" />
+      </inertial>
+    </link>
+    <joint name="${leg_name}_shoulder_gearbox" type="fixed">
+      <parent link="${leg_name}_upper_leg" />
+      <child link="${leg_name}_outer_gearbox" />
+      <origin xyz="0 -0.07 0" rpy="1.5707963267948963 0 0" />
     </joint>
     <link name="${leg_name}_upper_leg">
@@ -73,20 +111,20 @@
         <origin xyz="0 0 0.15" />
         <geometry>
-          <cylinder radius="0.055" length="0.3" />
-        </geometry>
-        <material name="purple">
-          <color rgba="0.43 0.27 0.52 1" />
-        </material>
-      </visual>
-      <collision>
-        <origin xyz="0 0 0.15" />
-        <geometry>
-          <cylinder radius="0.055" length="0.3" />
-        </geometry>
-      </collision>
-      <inertial>
-        <mass value="0.8" />
-        <inertia ixx="0.01" iyy="0.01" izz="0.01"
-                 ixy="0" ixz="0" iyz="0" />
+          <cylinder radius="0.038" length="0.3" />
+        </geometry>
+        <material name="purple">
+          <color rgba="0.43 0.27 0.52 1" />
+        </material>
+      </visual>
+      <collision>
+        <origin xyz="0 0 0.15" />
+        <geometry>
+          <cylinder radius="0.038" length="0.3" />
+        </geometry>
+      </collision>
+      <inertial>
+        <mass value="0.55" />
+        <inertia ixx="0.01" iyy="0.01" izz="0.01"
+          ixy="0" ixz="0" iyz="0" />
       </inertial>
     </link>
@@ -94,7 +132,8 @@
       <parent link="${leg_name}_upper_leg" />
       <child link="${leg_name}_lower_leg" />
-      <origin xyz="0 0 0.3" rpy="0 0 0" />
-      <axis xyz="0 1 0" />
-      <limit effort="200.0" velocity="2.0" lower="-1.57" upper="1.57" />
+      <origin xyz="0 0 0.3" rpy="0 ${knee_rot_off} 0" />
+      <axis xyz="${axis}" />
+      <limit effort="${effort}" velocity="${max_joint_velocity}" lower="${knee_lower_limit}"
+        upper="${knee_upper_limit}" />
     </joint>
     <link name="${leg_name}_lower_leg">
@@ -102,20 +141,77 @@
         <origin xyz="0 0 0.15" />
         <geometry>
-          <cylinder radius="0.035" length="0.3" />
-        </geometry>
-        <material name="purple">
-          <color rgba="0.43 0.27 0.52 1" />
-        </material>
-      </visual>
-      <collision>
-        <origin xyz="0 0 0.15" />
-        <geometry>
-          <cylinder radius="0.035" length="0.3" />
-        </geometry>
-      </collision>
-      <inertial>
-        <mass value="0.8" />
-        <inertia ixx="0.01" iyy="0.01" izz="0.01"
-                 ixy="0" ixz="0" iyz="0" />
+          <cylinder radius="0.026" length="0.3" />
+        </geometry>
+        <material name="purple">
+          <color rgba="0.43 0.27 0.52 1" />
+        </material>
+      </visual>
+      <collision>
+        <origin xyz="0 0 0.15" />
+        <geometry>
+          <cylinder radius="0.026" length="0.3" />
+        </geometry>
+      </collision>
+      <inertial>
+        <mass value="0.4" />
+        <inertia ixx="0.01" iyy="0.01" izz="0.01"
+          ixy="0" ixz="0" iyz="0" />
+      </inertial>
+    </link>
+    <joint name="${leg_name}_sock_connector" type="fixed">
+      <parent link="${leg_name}_lower_leg" />
+      <child link="${leg_name}_sock" />
+      <origin xyz="0 0 0.3" rpy="1.5707963267948966 0 0" />
+    </joint>
+    <link name="${leg_name}_sock">
+      <visual>
+        <origin xyz="0 0 0" />
+        <geometry>
+          <cylinder radius="0.030" length="0.025" />
+        </geometry>
+        <material name="kinda_blue">
+          <color rgba="0.27 0.27 0.52 1" />
+        </material>
+      </visual>
+      <visual>
+        <origin xyz="0 0 0.0125" />
+        <geometry>
+          <sphere radius="0.030" />
+        </geometry>
+        <material name="kinda_blue">
+          <color rgba="0.27 0.27 0.52 1" />
+        </material>
+      </visual>
+      <visual>
+        <origin xyz="0 0 -0.0125" />
+        <geometry>
+          <sphere radius="0.030" />
+        </geometry>
+        <material name="kinda_blue">
+          <color rgba="0.27 0.27 0.52 1" />
+        </material>
+      </visual>
+      <collision>
+        <origin xyz="0 0 0" />
+        <geometry>
+          <cylinder radius="0.030" length="0.025" />
+        </geometry>
+      </collision>
+      <collision>
+        <origin xyz="0 0 0.0125" />
+        <geometry>
+          <sphere radius="0.030" />
+        </geometry>
+      </collision>
+      <collision>
+        <origin xyz="0 0 -0.0125" />
+        <geometry>
+          <sphere radius="0.030" />
+        </geometry>
+      </collision>
+      <inertial>
+        <mass value="0.1" />
+        <inertia ixx="0.01" iyy="0.01" izz="0.01"
+          ixy="0" ixz="0" iyz="0" />
       </inertial>
     </link>
