Commit message: updated

File: cerberus_ws/install/cerberus_description/share/cerberus_description/urdf/cerbiboi.urdf.xacro (robot description, xacro)
@@ -2,6 +2,6 @@
 <robot xmlns:xacro="http://www.ros.org/wiki/xacro" name="Cerberus">
     <xacro:include filename="$(find cerberus_description)/urdf/leg_macro.xacro" />
-    <xacro:arg name="effort" default="55" />
-    <xacro:arg name="max_joint_velocity" default="1.0" />
+    <xacro:arg name="effort" default="40" />
+    <xacro:arg name="max_joint_velocity" default="2.0" />
     <!--
     <link name="world" />

File: cerberus_ws/install/cerberus_description/share/cerberus_description/urdf/leg_macro.xacro (robot description, xacro)
@@ -49,5 +49,5 @@
       <axis xyz="${axis}" />
       <limit effort="${effort}" velocity="${max_joint_velocity}" lower="-1.57" upper="1.57" />
-      <dynamics damping="0.9" friction="0.05" />
+      <dynamics damping="0.9" friction="0.02" />
     </joint>
     <link name="${leg_name}_gearbox_shoulder2">
@@ -81,5 +81,5 @@
       <limit effort="${effort}" velocity="${max_joint_velocity}" lower="${shoulder_lower_limit}"
         upper="${shoulder_upper_limit}" />
-        <dynamics damping="0.9" friction="0.05" />
+        <dynamics damping="0.9" friction="0.02" />
     </joint>
     <link name="${leg_name}_outer_gearbox">
@@ -141,5 +141,5 @@
       <limit effort="${effort}" velocity="${max_joint_velocity}" lower="${knee_lower_limit}"
         upper="${knee_upper_limit}" />
-      <dynamics damping="0.9" friction="0.05" />
+      <dynamics damping="0.9" friction="0.02" />
     </joint>
     <link name="${leg_name}_lower_leg">
