Commit message: updated urdf

File: cerberus_ws/src/cerberus/cerberus_description/urdf/cerberus.urdf (robot description, URDF)
Before this commit: robot Cerberus, 25 links, 24 joints
Links:
- removed link FL_sock
- removed link FR_sock
- removed link RL_sock
- removed link RR_sock
- added link FL_foot, mass 0.1; collision cylinder length=0.025 radius=0.030; collision sphere radius=0.030
- added link FR_foot, mass 0.1; collision cylinder length=0.025 radius=0.030; collision sphere radius=0.030
- added link RL_foot, mass 0.1; collision cylinder length=0.025 radius=0.030; collision sphere radius=0.030
- added link RR_foot, mass 0.1; collision cylinder length=0.025 radius=0.030; collision sphere radius=0.030
Joints:
- joint FL_calf_joint: limit lower=-0.5235987756 upper=1.047197551 effort=35 velocity=35 -> lower=-0.5235987756 upper=1.047197551 effort=45 velocity=45
- joint FL_hip_joint: limit lower=-1.57 upper=1.57 effort=35 velocity=35 -> lower=-1.57 upper=1.57 effort=45 velocity=45
- joint FL_thigh_joint: limit lower=-2.094395102 upper=1.047197551 effort=35 velocity=35 -> lower=-2.094395102 upper=1.047197551 effort=45 velocity=45
- joint FR_calf_joint: limit lower=-0.5235987756 upper=1.047197551 effort=35 velocity=35 -> lower=-0.5235987756 upper=1.047197551 effort=45 velocity=45
- joint FR_hip_joint: limit lower=-1.57 upper=1.57 effort=35 velocity=35 -> lower=-1.57 upper=1.57 effort=45 velocity=45
- joint FR_thigh_joint: limit lower=-2.094395102 upper=1.047197551 effort=35 velocity=35 -> lower=-2.094395102 upper=1.047197551 effort=45 velocity=45
- joint RL_calf_joint: limit lower=-0.5235987756 upper=1.047197551 effort=35 velocity=35 -> lower=-0.5235987756 upper=1.047197551 effort=45 velocity=45
- joint RL_hip_joint: limit lower=-1.57 upper=1.57 effort=35 velocity=35 -> lower=-1.57 upper=1.57 effort=45 velocity=45
- joint RL_thigh_joint: limit lower=-2.094395102 upper=1.047197551 effort=35 velocity=35 -> lower=-2.094395102 upper=1.047197551 effort=45 velocity=45
- joint RR_calf_joint: limit lower=-0.5235987756 upper=1.047197551 effort=35 velocity=35 -> lower=-0.5235987756 upper=1.047197551 effort=45 velocity=45
- joint RR_hip_joint: limit lower=-1.57 upper=1.57 effort=35 velocity=35 -> lower=-1.57 upper=1.57 effort=45 velocity=45
- joint RR_thigh_joint: limit lower=-2.094395102 upper=1.047197551 effort=35 velocity=35 -> lower=-2.094395102 upper=1.047197551 effort=45 velocity=45

File: cerberus_ws/src/cerberus/cerberus_description/urdf/cerbiboi.urdf.xacro (robot description, xacro)
@@ -2,5 +2,5 @@
 <robot xmlns:xacro="http://www.ros.org/wiki/xacro" name="Cerberus">
     <xacro:include filename="$(find cerberus_description)/urdf/leg_macro.xacro" />
-    <xacro:arg name="effort" default="35" />
+    <xacro:arg name="effort" default="45" />
     <xacro:arg name="max_joint_velocity" default="150.0" />
     <!--

File: cerberus_ws/src/cerberus/cerberus_description/urdf/leg_macro.xacro (robot description, xacro)
@@ -164,5 +164,5 @@
       <origin xyz="0 0 0.3" rpy="1.5707963267948966 0 0" />
     </joint>
-    <link name="${leg_name}_sock">
+    <link name="${leg_name}_foot">
       <visual>
         <origin xyz="0 0 0" />

Commit message: updated urdf

File: cerberus_ws/src/cerberus/cerberus_description/urdf/cerberus.urdf (robot description, URDF)
Before this commit: robot Cerberus, 25 links, 24 joints
Joints:
- joint FL_foot_fixed: child FL_sock -> FL_foot
- joint FR_foot_fixed: child FR_sock -> FR_foot
- joint RL_foot_fixed: child RL_sock -> RL_foot
- joint RR_foot_fixed: child RR_sock -> RR_foot

File: cerberus_ws/src/cerberus/cerberus_description/urdf/leg_macro.xacro (robot description, xacro)
@@ -161,5 +161,5 @@
     <joint name="${leg_name}_foot_fixed" type="fixed">
       <parent link="${leg_name}_lower_leg" />
-      <child link="${leg_name}_sock" />
+      <child link="${leg_name}_foot" />
       <origin xyz="0 0 0.3" rpy="1.5707963267948966 0 0" />
     </joint>

Commit message: updated urdf

File: cerberus_ws/src/cerberus/cerberus_description/urdf/cerberus.urdf (robot description, URDF)
Before this commit: robot Cerberus, 25 links, 24 joints
Joints:
- joint FL_foot_fixed: axis (none) -> 1 0 0; limit (none) -> lower=0 upper=0; type fixed -> revolute
- joint FR_foot_fixed: axis (none) -> 1 0 0; limit (none) -> lower=0 upper=0; type fixed -> revolute
- joint RL_foot_fixed: axis (none) -> 1 0 0; limit (none) -> lower=0 upper=0; type fixed -> revolute
- joint RR_foot_fixed: axis (none) -> 1 0 0; limit (none) -> lower=0 upper=0; type fixed -> revolute

File: cerberus_ws/src/cerberus/cerberus_description/urdf/leg_macro.xacro (robot description, xacro)
@@ -159,8 +159,11 @@
       </inertial>
     </link>
-    <joint name="${leg_name}_foot_fixed" type="fixed">
+    <joint name="${leg_name}_foot_fixed" type="revolute">
       <parent link="${leg_name}_lower_leg" />
       <child link="${leg_name}_foot" />
       <origin xyz="0 0 0.3" rpy="1.5707963267948966 0 0" />
+      <axis xyz="1 0 0" />
+      <limit lower="0"
+        upper="0" />
     </joint>
     <link name="${leg_name}_foot">

Commit message: updated urdf

File: cerberus_ws/src/cerberus/cerberus_description/urdf/cerberus.urdf (robot description, URDF)
Before this commit: robot Cerberus, 25 links, 24 joints
Links:
- added link imu_link, mass 0.01
Joints:
- added joint imu_joint: type fixed, parent base_link, child imu_link, origin xyz=0 0 0.1 rpy=0 0 0
- joint FL_calf_joint: limit lower=-0.5235987756 upper=1.047197551 effort=45 velocity=45 -> lower=-0.5235987756 upper=1.047197551 effort=55 velocity=1.0
- joint FL_foot_fixed: limit lower=0 upper=0 -> lower=0 upper=0 effort=0 velocity=0
- joint FL_hip_joint: limit lower=-1.57 upper=1.57 effort=45 velocity=45 -> lower=-1.57 upper=1.57 effort=55 velocity=1.0
- joint FL_thigh_joint: limit lower=-2.094395102 upper=1.047197551 effort=45 velocity=45 -> lower=-2.094395102 upper=1.047197551 effort=55 velocity=1.0
- joint FR_calf_joint: limit lower=-0.5235987756 upper=1.047197551 effort=45 velocity=45 -> lower=-0.5235987756 upper=1.047197551 effort=55 velocity=1.0
- joint FR_foot_fixed: limit lower=0 upper=0 -> lower=0 upper=0 effort=0 velocity=0
- joint FR_hip_joint: limit lower=-1.57 upper=1.57 effort=45 velocity=45 -> lower=-1.57 upper=1.57 effort=55 velocity=1.0
- joint FR_thigh_joint: limit lower=-2.094395102 upper=1.047197551 effort=45 velocity=45 -> lower=-2.094395102 upper=1.047197551 effort=55 velocity=1.0
- joint RL_calf_joint: limit lower=-0.5235987756 upper=1.047197551 effort=45 velocity=45 -> lower=-0.5235987756 upper=1.047197551 effort=55 velocity=1.0
- joint RL_foot_fixed: limit lower=0 upper=0 -> lower=0 upper=0 effort=0 velocity=0
- joint RL_hip_joint: limit lower=-1.57 upper=1.57 effort=45 velocity=45 -> lower=-1.57 upper=1.57 effort=55 velocity=1.0
- joint RL_thigh_joint: limit lower=-2.094395102 upper=1.047197551 effort=45 velocity=45 -> lower=-2.094395102 upper=1.047197551 effort=55 velocity=1.0
- joint RR_calf_joint: limit lower=-0.5235987756 upper=1.047197551 effort=45 velocity=45 -> lower=-0.5235987756 upper=1.047197551 effort=55 velocity=1.0
- joint RR_foot_fixed: limit lower=0 upper=0 -> lower=0 upper=0 effort=0 velocity=0
- joint RR_hip_joint: limit lower=-1.57 upper=1.57 effort=45 velocity=45 -> lower=-1.57 upper=1.57 effort=55 velocity=1.0
- joint RR_thigh_joint: limit lower=-2.094395102 upper=1.047197551 effort=45 velocity=45 -> lower=-2.094395102 upper=1.047197551 effort=55 velocity=1.0
