Commit message: updated launch files

File: cerberus_description/urdf/cerberus_odrive.urdf.xacro (robot description, xacro)
@@ -1,167 +1,155 @@
 <?xml version="1.0"?>
 <robot xmlns:xacro="http://www.ros.org/wiki/xacro" name="odrive_robot">
-  <!-- Arguments controlling whether each of the 12 joints is enabled -->
-  <xacro:arg name="enable_joint0"  default="false" />
-  <xacro:arg name="enable_joint1"  default="false" />
-  <xacro:arg name="enable_joint2"  default="false" />
-  <xacro:arg name="enable_joint3"  default="false" />
-  <xacro:arg name="enable_joint4"  default="false" />
-  <xacro:arg name="enable_joint5"  default="false" />
-  <xacro:arg name="enable_joint6"  default="false" />
-  <xacro:arg name="enable_joint7"  default="false" />
-  <xacro:arg name="enable_joint8"  default="false" />
-  <xacro:arg name="enable_joint9"  default="false" />
-  <xacro:arg name="enable_joint10" default="false" />
-  <xacro:arg name="enable_joint11" default="false" />
-  <!-- Arguments for up to 6 ODrive boards (2 axes each) -->
-  <xacro:arg name="odrive_1_serial" default="2081356E524B" />
-  <xacro:arg name="odrive_2_serial" default="20763599524B" />
-  <xacro:arg name="odrive_3_serial" default="000000000000" />
-  <xacro:arg name="odrive_4_serial" default="000000000000" />
-  <xacro:arg name="odrive_5_serial" default="000000000000" />
-  <xacro:arg name="odrive_6_serial" default="000000000000" />
-  <!-- Include your custom ODrive xacro definition that handles up to two axes -->
+  <xacro:arg name="enable_FL_hip_joint"  default="false" />
+  <xacro:arg name="enable_FR_hip_joint"  default="false" />
+  <xacro:arg name="enable_RL_hip_joint"  default="false" />
+  <xacro:arg name="enable_RR_hip_joint"  default="false" />
+  <xacro:arg name="enable_FL_thigh_joint"  default="false" />
+  <xacro:arg name="enable_FR_thigh_joint"  default="false" />
+  <xacro:arg name="enable_RL_thigh_joint"  default="false" />
+  <xacro:arg name="enable_RR_thigh_joint"  default="false" />
+  <xacro:arg name="enable_FL_calf_joint"  default="false" />
+  <xacro:arg name="enable_FR_calf_joint"  default="false" />
+  <xacro:arg name="enable_RL_calf_joint"  default="false" />
+  <xacro:arg name="enable_RR_calf_joint"  default="false" />
+  <xacro:arg name="front_hip_serial" default="20763599524B" />
+  <xacro:arg name="front_thigh_serial" default="2081356E524B" />
+  <xacro:arg name="front_calf_serial" default="205B39814D4D" />
+  <xacro:arg name="rear_hip_serial"  default="208339814D4D" />
+  <xacro:arg name="rear_thigh_serial" default="345735573033" />
+  <xacro:arg name="rear_calf_serial"  default="346035533033" />
   <xacro:include filename="$(find cerberus_description)/urdf/odrive.ros2_control.xacro" />
-  <!-- A world link to anchor everything -->
   <link name="world" />
-  <!-- Define 12 links and 12 joints, each optional behind an enable_jointN check -->
-  <xacro:if value="$(arg enable_joint0)">
-    <link name="link0" />
-    <joint name="joint0" type="continuous">
+  <xacro:if value="$(arg enable_FL_hip_joint)">
+    <link name="FL_hip_link" />
+    <joint name="FL_hip_joint" type="continuous">
       <parent link="world"/>
-      <child link="link0"/>
+      <child link="FL_hip_link"/>
       <axis xyz="0 0 1"/>
     </joint>
   </xacro:if>
-  <xacro:if value="$(arg enable_joint1)">
-    <link name="link1" />
-    <joint name="joint1" type="continuous">
+  <xacro:if value="$(arg enable_FR_hip_joint)">
+    <link name="FR_hip_link" />
+    <joint name="FR_hip_joint" type="continuous">
       <parent link="world"/>
-      <child link="link1"/>
+      <child link="FR_hip_link"/>
       <axis xyz="0 0 1"/>
     </joint>
   </xacro:if>
-  <xacro:if value="$(arg enable_joint2)">
-    <link name="link2" />
-    <joint name="joint2" type="continuous">
+  <xacro:if value="$(arg enable_RL_hip_joint)">
+    <link name="RL_hip_link" />
+    <joint name="RL_hip_joint" type="continuous">
       <parent link="world"/>
-      <child link="link2"/>
+      <child link="RL_hip_link"/>
       <axis xyz="0 0 1"/>
     </joint>
   </xacro:if>
-  <xacro:if value="$(arg enable_joint3)">
-    <link name="link3" />
-    <joint name="joint3" type="continuous">
+  <xacro:if value="$(arg enable_RR_hip_joint)">
+    <link name="RR_hip_link" />
+    <joint name="RR_hip_joint" type="continuous">
       <parent link="world"/>
-      <child link="link3"/>
+      <child link="RR_hip_link"/>
       <axis xyz="0 0 1"/>
     </joint>
   </xacro:if>
-  <xacro:if value="$(arg enable_joint4)">
-    <link name="link4" />
-    <joint name="joint4" type="continuous">
+  <xacro:if value="$(arg enable_FL_thigh_joint)">
+    <link name="FL_thigh_link" />
+    <joint name="FL_thigh_joint" type="continuous">
       <parent link="world"/>
-      <child link="link4"/>
+      <child link="FL_thigh_link"/>
       <axis xyz="0 0 1"/>
     </joint>
   </xacro:if>
-  <xacro:if value="$(arg enable_joint5)">
-    <link name="link5" />
-    <joint name="joint5" type="continuous">
+  <xacro:if value="$(arg enable_FR_thigh_joint)">
+    <link name="FR_thigh_link" />
+    <joint name="FR_thigh_joint" type="continuous">
       <parent link="world"/>
-      <child link="link5"/>
+      <child link="FR_thigh_link"/>
       <axis xyz="0 0 1"/>
     </joint>
   </xacro:if>
-  <xacro:if value="$(arg enable_joint6)">
-    <link name="link6" />
-    <joint name="joint6" type="continuous">
+  <xacro:if value="$(arg enable_RL_thigh_joint)">
+    <link name="RL_thigh_link" />
+    <joint name="RL_thigh_joint" type="continuous">
       <parent link="world"/>
-      <child link="link6"/>
+      <child link="RL_thigh_link"/>
       <axis xyz="0 0 1"/>
     </joint>
   </xacro:if>
-  <xacro:if value="$(arg enable_joint7)">
-    <link name="link7" />
-    <joint name="joint7" type="continuous">
+  <xacro:if value="$(arg enable_RR_thigh_joint)">
+    <link name="RR_thigh_link" />
+    <joint name="RR_thigh_joint" type="continuous">
       <parent link="world"/>
-      <child link="link7"/>
+      <child link="RR_thigh_link"/>
       <axis xyz="0 0 1"/>
     </joint>
   </xacro:if>
-  <xacro:if value="$(arg enable_joint8)">
-    <link name="link8" />
-    <joint name="joint8" type="continuous">
+  <xacro:if value="$(arg enable_FL_calf_joint)">
+    <link name="FL_calf_link" />
+    <joint name="FL_calf_joint" type="continuous">
       <parent link="world"/>
-      <child link="link8"/>
+      <child link="FL_calf_link"/>
       <axis xyz="0 0 1"/>
     </joint>
   </xacro:if>
-  <xacro:if value="$(arg enable_joint9)">
-    <link name="link9" />
-    <joint name="joint9" type="continuous">
+  <xacro:if value="$(arg enable_FR_calf_joint)">
+    <link name="FR_calf_link" />
+    <joint name="FR_calf_joint" type="continuous">
       <parent link="world"/>
-      <child link="link9"/>
+      <child link="FR_calf_link"/>
       <axis xyz="0 0 1"/>
     </joint>
   </xacro:if>
-  <xacro:if value="$(arg enable_joint10)">
-    <link name="link10" />
-    <joint name="joint10" type="continuous">
+  <xacro:if value="$(arg enable_RL_calf_joint)">
+    <link name="RL_calf_link" />
+    <joint name="RL_calf_joint" type="continuous">
       <parent link="world"/>
-      <child link="link10"/>
+      <child link="RL_calf_link"/>
       <axis xyz="0 0 1"/>
     </joint>
   </xacro:if>
-  <xacro:if value="$(arg enable_joint11)">
-    <link name="link11" />
-    <joint name="joint11" type="continuous">
+  <xacro:if value="$(arg enable_RR_calf_joint)">
+    <link name="RR_calf_link" />
+    <joint name="RR_calf_joint" type="continuous">
       <parent link="world"/>
-      <child link="link11"/>
+      <child link="RR_calf_link"/>
       <axis xyz="0 0 1"/>
     </joint>
   </xacro:if>
-  <!-- Now define 6 possible ODrive boards, each controlling 2 joints -->
-  <!-- ODrive #1: controls joint0 and joint1 -->
   <xacro:odrive_ros2_control
-    name="odrive1_ros2_control"
+    name="front_hip_ros2_control"
     sensor_name="odrv0"
-    serial_number="$(arg odrive_1_serial)"
-    joint0_name="joint0" enable_joint0="$(arg enable_joint0)"
-    joint1_name="joint1" enable_joint1="$(arg enable_joint1)" />
-  <!-- ODrive #2: controls joint2 and joint3 -->
+    serial_number="$(arg front_hip_serial)"
+    joint0_name="FL_hip_joint" enable_joint0="$(arg enable_FL_hip_joint)"
+    joint1_name="FR_hip_joint" enable_joint1="$(arg enable_FR_hip_joint)" />
   <xacro:odrive_ros2_control
-    name="odrive2_ros2_control"
+    name="front_thigh_ros2_control"
     sensor_name="odrv1"
-    serial_number="$(arg odrive_2_serial)"
-    joint0_name="joint2" enable_joint0="$(arg enable_joint2)"
-    joint1_name="joint3" enable_joint1="$(arg enable_joint3)" />
-  <!-- ODrive #3: controls joint4 and joint5 -->
+    serial_number="$(arg front_thigh_serial)"
+    joint0_name="FL_thigh_joint" enable_joint0="$(arg enable_FL_thigh_joint)"
+    joint1_name="FR_thigh_joint" enable_joint1="$(arg enable_FR_thigh_joint)" />
   <xacro:odrive_ros2_control
-    name="odrive3_ros2_control"
+    name="front_calf_ros2_control"
     sensor_name="odrv2"
-    serial_number="$(arg odrive_3_serial)"
-    joint0_name="joint4" enable_joint0="$(arg enable_joint4)"
-    joint1_name="joint5" enable_joint1="$(arg enable_joint5)" />
-  <!-- ODrive #4: controls joint6 and joint7 -->
+    serial_number="$(arg front_calf_serial)"
+    joint0_name="FL_calf_joint" enable_joint0="$(arg enable_FL_calf_joint)"
+    joint1_name="FR_calf_joint" enable_joint1="$(arg enable_FR_calf_joint)" />
   <xacro:odrive_ros2_control
-    name="odrive4_ros2_control"
+    name="rear_hip_ros2_control"
     sensor_name="odrv3"
-    serial_number="$(arg odrive_4_serial)"
-    joint0_name="joint6" enable_joint0="$(arg enable_joint6)"
-    joint1_name="joint7" enable_joint1="$(arg enable_joint7)" />
-  <!-- ODrive #5: controls joint8 and joint9 -->
+    serial_number="$(arg rear_hip_serial)"
+    joint0_name="RL_hip_joint" enable_joint0="$(arg enable_RL_hip_joint)"
+    joint1_name="RR_hip_joint" enable_joint1="$(arg enable_RR_hip_joint)" />
   <xacro:odrive_ros2_control
-    name="odrive5_ros2_control"
+    name="rear_thigh_ros2_control"
     sensor_name="odrv4"
-    serial_number="$(arg odrive_5_serial)"
-    joint0_name="joint8" enable_joint0="$(arg enable_joint8)"
-    joint1_name="joint9" enable_joint1="$(arg enable_joint9)" />
-  <!-- ODrive #6: controls joint10 and joint11 -->
+    serial_number="$(arg rear_thigh_serial)"
+    joint0_name="RL_thigh_joint" enable_joint0="$(arg enable_RL_thigh_joint)"
+    joint1_name="RR_thigh_joint" enable_joint1="$(arg enable_RR_thigh_joint)" />
   <xacro:odrive_ros2_control
-    name="odrive6_ros2_control"
+    name="rear_calf_ros2_control"
     sensor_name="odrv5"
-    serial_number="$(arg odrive_6_serial)"
-    joint0_name="joint10" enable_joint0="$(arg enable_joint10)"
-    joint1_name="joint11" enable_joint1="$(arg enable_joint11)" />
+    serial_number="$(arg rear_calf_serial)"
+    joint0_name="RL_calf_joint" enable_joint0="$(arg enable_RL_calf_joint)"
+    joint1_name="RR_calf_joint" enable_joint1="$(arg enable_RR_calf_joint)" />
 </robot>
