Commit message: updated controls

File: cerberus_description/urdf/cerbiboi.urdf.xacro (robot description, xacro)
@@ -2,6 +2,6 @@
 <robot xmlns:xacro="http://www.ros.org/wiki/xacro" name="Cerberus">
     <xacro:include filename="$(find cerberus_description)/urdf/leg_macro.xacro" />
-    <xacro:arg name="effort" default="40" />
-    <xacro:arg name="max_joint_velocity" default="2.0" />
+    <xacro:arg name="effort" default="80" />
+    <xacro:arg name="max_joint_velocity" default="5.00" />
     <!--
     <link name="world" />
@@ -176,4 +176,5 @@
             <command_interface name="position" />
             <command_interface name="velocity" />
+            <command_interface name="effort" />
             <state_interface name="position" />
             <state_interface name="velocity" />
@@ -183,4 +184,5 @@
             <command_interface name="position" />
             <command_interface name="velocity" />
+            <command_interface name="effort" />
             <state_interface name="position" />
             <state_interface name="velocity" />
@@ -190,4 +192,5 @@
             <command_interface name="position" />
             <command_interface name="velocity" />
+            <command_interface name="effort" />
             <state_interface name="position" />
             <state_interface name="velocity" />
@@ -197,4 +200,5 @@
             <command_interface name="position" />
             <command_interface name="velocity" />
+            <command_interface name="effort" />
             <state_interface name="position" />
             <state_interface name="velocity" />
@@ -204,4 +208,5 @@
             <command_interface name="position" />
             <command_interface name="velocity" />
+            <command_interface name="effort" />
             <state_interface name="position" />
             <state_interface name="velocity" />
@@ -211,4 +216,5 @@
             <command_interface name="position" />
             <command_interface name="velocity" />
+            <command_interface name="effort" />
             <state_interface name="position" />
             <state_interface name="velocity" />
@@ -218,4 +224,5 @@
             <command_interface name="position" />
             <command_interface name="velocity" />
+            <command_interface name="effort" />
             <state_interface name="position" />
             <state_interface name="velocity" />
@@ -225,4 +232,5 @@
             <command_interface name="position" />
             <command_interface name="velocity" />
+            <command_interface name="effort" />
             <state_interface name="position" />
             <state_interface name="velocity" />
@@ -232,4 +240,5 @@
             <command_interface name="position" />
             <command_interface name="velocity" />
+            <command_interface name="effort" />
             <state_interface name="position" />
             <state_interface name="velocity" />
@@ -239,4 +248,5 @@
             <command_interface name="position" />
             <command_interface name="velocity" />
+            <command_interface name="effort" />
             <state_interface name="position" />
             <state_interface name="velocity" />
@@ -246,4 +256,5 @@
             <command_interface name="position" />
             <command_interface name="velocity" />
+            <command_interface name="effort" />
             <state_interface name="position" />
             <state_interface name="velocity" />
@@ -253,4 +264,5 @@
             <command_interface name="position" />
             <command_interface name="velocity" />
+            <command_interface name="effort" />
             <state_interface name="position" />
             <state_interface name="velocity" />

File: cerberus_description/urdf/leg_macro.xacro (robot description, xacro)
@@ -49,5 +49,5 @@
       <axis xyz="${axis}" />
       <limit effort="${effort}" velocity="${max_joint_velocity}" lower="-1.57" upper="1.57" />
-      <dynamics damping="0.9" friction="0.02" />
+      <dynamics damping="0.001" friction="1"/>
     </joint>
     <link name="${leg_name}_gearbox_shoulder2">
@@ -81,6 +81,6 @@
       <limit effort="${effort}" velocity="${max_joint_velocity}" lower="${shoulder_lower_limit}"
         upper="${shoulder_upper_limit}" />
-        <dynamics damping="0.9" friction="0.02" />
-    </joint>
+        <dynamics damping="0.001" friction="1"/>
+      </joint>
     <link name="${leg_name}_outer_gearbox">
       <visual>
@@ -141,6 +141,6 @@
       <limit effort="${effort}" velocity="${max_joint_velocity}" lower="${knee_lower_limit}"
         upper="${knee_upper_limit}" />
-      <dynamics damping="0.9" friction="0.02" />
-    </joint>
+        <dynamics damping="0.001" friction="1"/>
+      </joint>
     <link name="${leg_name}_lower_leg">
       <visual>

Commit message: updated software

File: cerberus_description/urdf/cerbiboi.urdf.xacro (robot description, xacro)
@@ -2,6 +2,6 @@
 <robot xmlns:xacro="http://www.ros.org/wiki/xacro" name="Cerberus">
     <xacro:include filename="$(find cerberus_description)/urdf/leg_macro.xacro" />
-    <xacro:arg name="effort" default="80" />
-    <xacro:arg name="max_joint_velocity" default="5.00" />
+    <xacro:arg name="effort" default="60" />
+    <xacro:arg name="max_joint_velocity" default="1.200" />
     <!--
     <link name="world" />
@@ -42,5 +42,5 @@
         <inertial>
             <mass value="5.0" />
-            <inertia ixx="0.1010416667" iyy="0.04980166667" izz="0.1175"
+            <inertia ixx="0.04980166667" iyy="0.1010416667" izz="0.1175"
                 ixy="0.0" ixz="0.0" iyz="0.0" />
         </inertial>
@@ -176,5 +176,4 @@
             <command_interface name="position" />
             <command_interface name="velocity" />
-            <command_interface name="effort" />
             <state_interface name="position" />
             <state_interface name="velocity" />
@@ -184,5 +183,4 @@
             <command_interface name="position" />
             <command_interface name="velocity" />
-            <command_interface name="effort" />
             <state_interface name="position" />
             <state_interface name="velocity" />
@@ -192,5 +190,4 @@
             <command_interface name="position" />
             <command_interface name="velocity" />
-            <command_interface name="effort" />
             <state_interface name="position" />
             <state_interface name="velocity" />
@@ -200,5 +197,4 @@
             <command_interface name="position" />
             <command_interface name="velocity" />
-            <command_interface name="effort" />
             <state_interface name="position" />
             <state_interface name="velocity" />
@@ -208,5 +204,4 @@
             <command_interface name="position" />
             <command_interface name="velocity" />
-            <command_interface name="effort" />
             <state_interface name="position" />
             <state_interface name="velocity" />
@@ -216,5 +211,4 @@
             <command_interface name="position" />
             <command_interface name="velocity" />
-            <command_interface name="effort" />
             <state_interface name="position" />
             <state_interface name="velocity" />
@@ -224,5 +218,4 @@
             <command_interface name="position" />
             <command_interface name="velocity" />
-            <command_interface name="effort" />
             <state_interface name="position" />
             <state_interface name="velocity" />
@@ -232,5 +225,4 @@
             <command_interface name="position" />
             <command_interface name="velocity" />
-            <command_interface name="effort" />
             <state_interface name="position" />
             <state_interface name="velocity" />
@@ -240,5 +232,4 @@
             <command_interface name="position" />
             <command_interface name="velocity" />
-            <command_interface name="effort" />
             <state_interface name="position" />
             <state_interface name="velocity" />
@@ -248,5 +239,4 @@
             <command_interface name="position" />
             <command_interface name="velocity" />
-            <command_interface name="effort" />
             <state_interface name="position" />
             <state_interface name="velocity" />
@@ -256,5 +246,4 @@
             <command_interface name="position" />
             <command_interface name="velocity" />
-            <command_interface name="effort" />
             <state_interface name="position" />
             <state_interface name="velocity" />
@@ -264,5 +253,4 @@
             <command_interface name="position" />
             <command_interface name="velocity" />
-            <command_interface name="effort" />
             <state_interface name="position" />
             <state_interface name="velocity" />
